File: sensors.kicad_sch (KiCad schematic)
At the start: 5 parts, among them U2 LIS2MDL

Commit message: Add files via upload
Parts:
- added C? (x2): 100 nF, symbol Device:C
- added U?: LSM6DSOX, symbol imu:LSM6DSOX
- renumbered C3 to C?, C2 to C?, C1 to C?, C4 to C?, U2 to U?
Connections:
- net +3.3V: now also C?.1, C?.1, U?.5 (VDDIO), U?.8 (VDD)
- net GND: now also C?.2, C?.2, U?.6 (GND), U?.7 (GND)
- net MISO: now also U?.1 (SDO/SA0)
- net MOSI: now also U?.14 (SDA)
- net SCK: now also U?.13 (SCL)
- new net IMU_CS: U?.12 (CS)
- new net IMU_INT1: U?.4 (INT1)
- no-connect marks 0 -> 5

Commit message: Add files via upload
Parts:
- C1, C2, C3, C4, C5, C6: renamed from C?; footprint (none) -> Capacitor_SMD:C_0201_0603Metric
- U3: renamed from U?; footprint (none) -> imu_footprint:PQFN50P250X300X86-14N
- gave numbers to parts that had none: 1
Changed lines of the file:
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@@
 		(on_board yes)
 		(dnp no)
-		(property "Reference" "C?"
+		(property "Reference" "C5"
 			(at 97.282 86.868 90)
 			(effects
@@
 			)
 		)
-		(property "Footprint" ""
+		(property "Footprint" "Capacitor_SMD:C_0201_0603Metric"
 			(at 92.71 89.2048 0)
 			(effects
@@
 				)
 			)
-			(project "flight-controller-basic"
-				(path "/e04fbe87-dc7c-407c-abef-b71ed1bbe06a/15ccaa96-ad63-4a4d-bfcd-1e00695c7116"
-					(reference "C?")
+			(project "sensors"
+				(path "/e04fbe87-dc7c-407c-abef-b71ed1bbe06a/26da8c72-585c-4186-816d-b3c1acee8ee0"
+					(reference "C5")
 					(unit 1)
 				)
@@
 		(on_board yes)
 		(dnp no)
-		(property "Reference" "C?"
+		(property "Reference" "C6"
 			(at 98.298 94.488 90)
 			(effects
@@
 			)
 		)
-		(property "Footprint" ""
+		(property "Footprint" "Capacitor_SMD:C_0201_0603Metric"
 			(at 92.71 94.2848 0)
 			(effects
@@
 				)
 			)
-			(project "flight-controller-basic"
-				(path "/e04fbe87-dc7c-407c-abef-b71ed1bbe06a/15ccaa96-ad63-4a4d-bfcd-1e00695c7116"
-					(reference "C?")
+			(project "sensors"
+				(path "/e04fbe87-dc7c-407c-abef-b71ed1bbe06a/26da8c72-585c-4186-816d-b3c1acee8ee0"
+					(reference "C6")
 					(unit 1)
 				)
@@
 		(dnp no)
 		(fields_autoplaced yes)
-		(property "Reference" "#PWR?"
+		(property "Reference" "#PWR06"
 			(at 83.82 88.9 0)
 			(effects
@@
 				)
 			)
-			(project "flight-controller-basic"
-				(path "/e04fbe87-dc7c-407c-abef-b71ed1bbe06a/15ccaa96-ad63-4a4d-bfcd-1e00695c7116"
-					(reference "#PWR?")
+			(project "sensors"
+				(path "/e04fbe87-dc7c-407c-abef-b71ed1bbe06a/26da8c72-585c-4186-816d-b3c1acee8ee0"
+					(reference "#PWR06")
 					(unit 1)
 				)
@@
 		(on_board yes)
 		(dnp no)
-		(property "Reference" "C?"
+		(property "Reference" "C2"
 			(at 90.17 38.354 90)
 			(effects
@@
 			)
 		)
-		(property "Footprint" ""
+		(property "Footprint" "Capacitor_SMD:C_0201_0603Metric"
 			(at 91.44 38.4048 0)
 			(effects
@@
 				)
 			)
-			(project "flight-controller-basic"
-				(path "/e04fbe87-dc7c-407c-abef-b71ed1bbe06a/15ccaa96-ad63-4a4d-bfcd-1e00695c7116"
-					(reference "C?")
+			(project "sensors"
+				(path "/e04fbe87-dc7c-407c-abef-b71ed1bbe06a/26da8c72-585c-4186-816d-b3c1acee8ee0"
+					(reference "C2")
 					(unit 1)
 				)
@@
 		(dnp no)
 		(fields_autoplaced yes)
-		(property "Reference" "#PWR?"
+		(property "Reference" "#PWR07"
 			(at 91.44 64.77 0)
 			(effects
@@
 				)
 			)
-			(project "flight-controller-basic"
-				(path "/e04fbe87-dc7c-407c-abef-b71ed1bbe06a/15ccaa96-ad63-4a4d-bfcd-1e00695c7116"
-					(reference "#PWR?")
+			(project "sensors"
+				(path "/e04fbe87-dc7c-407c-abef-b71ed1bbe06a/26da8c72-585c-4186-816d-b3c1acee8ee0"
+					(reference "#PWR07")
 					(unit 1)
 				)
@@
 		(on_board yes)
 		(dnp no)
-		(property "Reference" "C?"
+		(property "Reference" "C1"
 			(at 89.154 33.528 90)
 			(effects
@@
 			)
 		)
-		(property "Footprint" ""
+		(property "Footprint" "Capacitor_SMD:C_0201_0603Metric"
 			(at 87.63 34.29 0)
 			(effects
@@
 				)
 			)
-			(project "flight-controller-basic"
-				(path "/e04fbe87-dc7c-407c-abef-b71ed1bbe06a/15ccaa96-ad63-4a4d-bfcd-1e00695c7116"
-					(reference "C?")
+			(project "sensors"
+				(path "/e04fbe87-dc7c-407c-abef-b71ed1bbe06a/26da8c72-585c-4186-816d-b3c1acee8ee0"
+					(reference "C1")
 					(unit 1)
 				)
@@
 		(dnp no)
 		(fields_autoplaced yes)
-		(property "Reference" "#PWR?"
+		(property "Reference" "#PWR08"
 			(at 92.71 127 0)
 			(effects
@@
 				)
 			)
-			(project "flight-controller-basic"
-				(path "/e04fbe87-dc7c-407c-abef-b71ed1bbe06a/15ccaa96-ad63-4a4d-bfcd-1e00695c7116"
-					(reference "#PWR?")
+			(project "sensors"
+				(path "/e04fbe87-dc7c-407c-abef-b71ed1bbe06a/26da8c72-585c-4186-816d-b3c1acee8ee0"
+					(reference "#PWR08")
 					(unit 1)
 				)
@@
 		(on_board yes)
 		(dnp no)
-		(property "Reference" "C?"
+		(property "Reference" "C4"
 			(at 89.916 49.784 90)
 			(effects
@@
 			)
 		)
-		(property "Footprint" ""
+		(property "Footprint" "Capacitor_SMD:C_0201_0603Metric"
 			(at 91.44 49.8348 0)
 			(effects
@@
 				)
 			)
-			(project "flight-controller-basic"
-				(path "/e04fbe87-dc7c-407c-abef-b71ed1bbe06a/15ccaa96-ad63-4a4d-bfcd-1e00695c7116"
-					(reference "C?")
+			(project "sensors"
+				(path "/e04fbe87-dc7c-407c-abef-b71ed1bbe06a/26da8c72-585c-4186-816d-b3c1acee8ee0"
+					(reference "C4")
 					(unit 1)
 				)
@@
 		(on_board yes)
 		(dnp no)
-		(property "Reference" "U?"
+		(property "Reference" "U4"
 			(at 74.93 35.814 0)
 			(effects
@@
 				)
 			)
-			(project "flight-controller-basic"
-				(path "/e04fbe87-dc7c-407c-abef-b71ed1bbe06a/15ccaa96-ad63-4a4d-bfcd-1e00695c7116"
-					(reference "U?")
+			(project "sensors"
+				(path "/e04fbe87-dc7c-407c-abef-b71ed1bbe06a/26da8c72-585c-4186-816d-b3c1acee8ee0"
+					(reference "U4")
 					(unit 1)
 				)
@@
 		(dnp no)
 		(fields_autoplaced yes)
-		(property "Reference" "U?"
+		(property "Reference" "U3"
 			(at 66.04 85.09 0)
 			(effects
@@
 			)
 		)
-		(property "Footprint" ""
+		(property "Footprint" "imu_footprint:PQFN50P250X300X86-14N"
 			(at 66.04 105.41 0)
 			(effects
@@
 				)
 			)
-			(project "flight-controller-basic"
-				(path "/e04fbe87-dc7c-407c-abef-b71ed1bbe06a/15ccaa96-ad63-4a4d-bfcd-1e00695c7116"
-					(reference "U?")
+			(project "sensors"
+				(path "/e04fbe87-dc7c-407c-abef-b71ed1bbe06a/26da8c72-585c-4186-816d-b3c1acee8ee0"
+					(reference "U3")
 					(unit 1)
 				)
@@
 		(on_board yes)
 		(dnp no)
-		(property "Reference" "C?"
+		(property "Reference" "C3"
 			(at 90.17 43.688 90)
 			(effects
@@
 			)
 		)
-		(property "Footprint" ""
+		(property "Footprint" "Capacitor_SMD:C_0201_0603Metric"
 			(at 91.44 43.4848 0)
 			(effects
@@
 				)
 			)
-			(project "flight-controller-basic"
-				(path "/e04fbe87-dc7c-407c-abef-b71ed1bbe06a/15ccaa96-ad63-4a4d-bfcd-1e00695c7116"
-					(reference "C?")
+			(project "sensors"
+				(path "/e04fbe87-dc7c-407c-abef-b71ed1bbe06a/26da8c72-585c-4186-816d-b3c1acee8ee0"
+					(reference "C3")
 					(unit 1)
 				)
@@
 		(dnp no)
 		(fields_autoplaced yes)
-		(property "Reference" "#PWR?"
+		(property "Reference" "#PWR05"
 			(at 82.55 35.56 0)
 			(effects
@@
 				)
 			)
-			(project "flight-controller-basic"
-				(path "/e04fbe87-dc7c-407c-abef-b71ed1bbe06a/15ccaa96-ad63-4a4d-bfcd-1e00695c7116"
-					(reference "#PWR?")
-					(unit 1)
-				)
-			)
-		)
-	)
-	(sheet_instances
-		(path "/"
-			(page "1")
-		)
-	)
-	(embedded_fonts no)
+			(project "sensors"
+				(path "/e04fbe87-dc7c-407c-abef-b71ed1bbe06a/26da8c72-585c-4186-816d-b3c1acee8ee0"
+					(reference "#PWR05")
+					(unit 1)
+				)
+			)
+		)
+	)
 )

Commit message: Add files via upload
Parts:
- added C10, C9: C, Capacitor_SMD:C_0201_0603Metric, symbol Device:C
- added U7: LPS22DFTR, QFN_22DFTR_STM, symbol New_Library:LPS22DFTR
Connections:
- net GND: now also C10.1, C10.2, C9.1, C9.2, U7.1 (Vdd_IO), U7.10 (VDD), U7.3 (RES), U7.8 (GND_IO), U7.9 (GND)
- net MISO: now also U7.5 (SDO/SA0)
- net MOSI: now also U7.4 (SDA/SDI/SDISDO)
- net SCK: now also U7.2 (SCL/SPC)
- new net BAR_CS: U7.6 (CS)
- new net BAR_INT: U7.7 (INT_DRDY)
