File: bomboclat-barometer.kicad_sch (KiCad schematic)
At the start: 4 parts, among them J1 Conn_01x05_Pin, U1 LPS22DFTR

Commit message: Add files via upload
Parts:
- removed J1: Conn_01x05_Pin, symbol Connector:Conn_01x05_Pin
- C7: renamed from C1; footprint (none) -> Capacitor_SMD:C_0201_0603Metric
- C8: renamed from C2; footprint (none) -> Capacitor_SMD:C_0201_0603Metric
- renumbered U1 to U5
Connections:
- net GND: no longer U5.5 (SDO/SA0), U5.6 (CS)
- net INT renamed BAR_INT
- net SCL renamed SCK
- net SDA renamed MOSI
- new net BAR_CS: U5.6 (CS)
- new net MISO: U5.5 (SDO/SA0)
