File: flight-controller-basic.kicad_sch (KiCad schematic)
At the start: 0 parts

Commit message: Add files via upload
pls work
Other:
- added sheet GPS (C:/Users/omn08/Downloads/omnia_FC_2026/IMU_FC_G/GP_GPS/GP_GPS.kicad_sch)
- added sheet SENSORS (sensors.kicad_sch)
- added sheet USB-C (FC_USB-C_G/FC_USB-C_G.kicad_sch)
Changed lines of the file:
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@@
 	(paper "A4")
+	(sheet
+		(at 34.29 100.33)
+		(size 29.21 26.67)
+		(exclude_from_sim no)
+		(in_bom yes)
+		(on_board yes)
+		(dnp no)
+		(fields_autoplaced yes)
+		(stroke
+			(width 0.1524)
+			(type solid)
+		)
+		(fill
+			(color 0 0 0 0.0000)
+		)
+		(property "Sheetname" "SENSORS"
+			(at 34.29 99.6184 0)
+			(effects
+				(font
+					(size 1.27 1.27)
+				)
+				(justify left bottom)
+			)
+		)
+		(property "Sheetfile" "sensors.kicad_sch"
+			(at 34.29 127.5846 0)
+			(effects
+				(font
+					(size 1.27 1.27)
+				)
+				(justify left top)
+			)
+		)
+		(instances
+			(project "flight-controller-basic"
+				(path "/e04fbe87-dc7c-407c-abef-b71ed1bbe06a"
+					(page "4")
+				)
+			)
+		)
+	)
 	(sheet
 		(at 34.29 34.29)
@@
 				)
 			)
+		)
+	)
+	(sheet
+		(at 34.29 66.04)
+		(size 29.21 27.94)
+		(exclude_from_sim no)
+		(in_bom yes)
+		(on_board yes)
+		(dnp no)
+		(fields_autoplaced yes)
+		(stroke
+			(width 0.1524)
+			(type solid)
+		)
+		(fill
+			(color 0 0 0 0.0000)
+		)
+		(property "Sheetname" "GPS"
+			(at 34.29 65.3284 0)
+			(effects
+				(font
+					(size 1.27 1.27)
+				)
+				(justify left bottom)
+			)
+		)
+		(property "Sheetfile" "C:/Users/omn08/Downloads/omnia_FC_2026/IMU_FC_G/GP_GPS/GP_GPS.kicad_sch"
+			(at 34.29 94.5646 0)
+			(effects
+				(font
+					(size 1.27 1.27)
+				)
+				(justify left top)
+			)
+		)
+		(instances
+			(project "flight-controller-basic"
+				(path "/e04fbe87-dc7c-407c-abef-b71ed1bbe06a"
+					(page "3")
+				)
+			)
+		)
+	)
+	(sheet
+		(at 77.47 33.02)
+		(size 29.21 25.4)
+		(exclude_from_sim no)
+		(in_bom yes)
+		(on_board yes)
+		(dnp no)
+		(fields_autoplaced yes)
+		(stroke
+			(width 0.1524)
+			(type solid)
+		)
+		(fill
+			(color 0 0 0 0.0000)
+		)
+		(property "Sheetname" "USB-C"
+			(at 77.47 32.3084 0)
+			(effects
+				(font
+					(size 1.27 1.27)
+				)
+				(justify left bottom)
+			)
+		)
+		(property "Sheetfile" "FC_USB-C_G/FC_USB-C_G.kicad_sch"
+			(at 77.47 59.0046 0)
+			(effects
+				(font
+					(size 1.27 1.27)
+				)
+				(justify left top)
+			)
+		)
+		(instances
+			(project "flight-controller-basic"
+				(path "/e04fbe87-dc7c-407c-abef-b71ed1bbe06a"
+					(page "5")
+				)
+			)

Commit message: Add files via upload
Other:
- added sheet BARO (bomboclat-barometer.kicad_sch)
- added sheet RADIO (RADIO_G/RADIO_G.kicad_sch)
Changed lines of the file:
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@@
+	)
+	(sheet
+		(at 77.47 64.77)
+		(size 29.21 24.13)
+		(exclude_from_sim no)
+		(in_bom yes)
+		(on_board yes)
+		(dnp no)
+		(fields_autoplaced yes)
+		(stroke
+			(width 0.1524)
+			(type solid)
+		)
+		(fill
+			(color 0 0 0 0.0000)
+		)
+		(property "Sheetname" "BARO"
+			(at 77.47 64.0584 0)
+			(effects
+				(font
+					(size 1.27 1.27)
+				)
+				(justify left bottom)
+			)
+		)
+		(property "Sheetfile" "bomboclat-barometer.kicad_sch"
+			(at 77.47 89.4846 0)
+			(effects
+				(font
+					(size 1.27 1.27)
+				)
+				(justify left top)
+			)
+		)
+		(instances
+			(project "flight-controller-basic"
+				(path "/e04fbe87-dc7c-407c-abef-b71ed1bbe06a"
+					(page "6")
+				)
+			)
+		)
+	)
+	(sheet
+		(at 77.47 102.87)
+		(size 31.75 24.13)
+		(exclude_from_sim no)
+		(in_bom yes)
+		(on_board yes)
+		(dnp no)
+		(fields_autoplaced yes)
+		(stroke
+			(width 0.1524)
+			(type solid)
+		)
+		(fill
+			(color 0 0 0 0.0000)
+		)
+		(property "Sheetname" "RADIO"
+			(at 77.47 102.1584 0)
+			(effects
+				(font
+					(size 1.27 1.27)
+				)
+				(justify left bottom)
+			)
+		)
+		(property "Sheetfile" "RADIO_G/RADIO_G.kicad_sch"
+			(at 77.47 127.5846 0)
+			(effects
+				(font
+					(size 1.27 1.27)
+				)
+				(justify left top)
+			)
+		)
+		(instances
+			(project "flight-controller-basic"
+				(path "/e04fbe87-dc7c-407c-abef-b71ed1bbe06a"
+					(page "7")
+				)
+			)
+		)
 	)
 	(sheet

Commit message: Add files via upload
Other:
- removed sheet BARO
Changed lines of the file:
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@@
 	)
 	(sheet
-		(at 77.47 64.77)
-		(size 29.21 24.13)
-		(exclude_from_sim no)
-		(in_bom yes)
-		(on_board yes)
-		(dnp no)
-		(fields_autoplaced yes)
-		(stroke
-			(width 0.1524)
-			(type solid)
-		)
-		(fill
-			(color 0 0 0 0.0000)
-		)
-		(property "Sheetname" "BARO"
-			(at 77.47 64.0584 0)
-			(effects
-				(font
-					(size 1.27 1.27)
-				)
-				(justify left bottom)
-			)
-		)
-		(property "Sheetfile" "bomboclat-barometer.kicad_sch"
-			(at 77.47 89.4846 0)
-			(effects
-				(font
-					(size 1.27 1.27)
-				)
-				(justify left top)
-			)
-		)
-		(instances
-			(project "flight-controller-basic"
-				(path "/e04fbe87-dc7c-407c-abef-b71ed1bbe06a"
-					(page "6")
-				)
-			)
-		)
-	)
-	(sheet
-		(at 77.47 102.87)
+		(at 77.47 66.04)
 		(size 31.75 24.13)
 		(exclude_from_sim no)
@@
 		)
 		(property "Sheetname" "RADIO"
-			(at 77.47 102.1584 0)
+			(at 77.47 65.3284 0)
 			(effects
 				(font
@@
 		)
 		(property "Sheetfile" "RADIO_G/RADIO_G.kicad_sch"
-			(at 77.47 127.5846 0)
+			(at 77.47 90.7546 0)
 			(effects
 				(font
