File: flight-controller-basic.kicad_sch (KiCad schematic)
At the start: 0 parts

Commit message: Added the Sheet for the SD card and started the schematic.
Other:
- added sheet SD (basic_flight_controller_SD.kicad_sch)
Changed lines of the file:
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@@
 	(paper "A4")
+	(sheet
+		(at 77.47 100.33)
+		(size 30.48 26.67)
+		(exclude_from_sim no)
+		(in_bom yes)
+		(on_board yes)
+		(dnp no)
+		(fields_autoplaced yes)
+		(stroke
+			(width 0.1524)
+			(type solid)
+		)
+		(fill
+			(color 0 0 0 0.0000)
+		)
+		(property "Sheetname" "SD"
+			(at 77.47 99.6184 0)
+			(effects
+				(font
+					(size 1.27 1.27)
+				)
+				(justify left bottom)
+			)
+		)
+		(property "Sheetfile" "basic_flight_controller_SD.kicad_sch"
+			(at 77.47 127.5846 0)
+			(effects
+				(font
+					(size 1.27 1.27)
+				)
+				(justify left top)
+			)
+		)
+		(instances
+			(project "flight-controller-basic"
+				(path "/e04fbe87-dc7c-407c-abef-b71ed1bbe06a"
+					(page "7")
+				)
+			)
+		)
+	)
 	(sheet
 		(at 34.29 100.33)
@@
 			(project "flight-controller-basic"
 				(path "/e04fbe87-dc7c-407c-abef-b71ed1bbe06a"
-					(page "7")
+					(page "6")
 				)
 			)

Commit message: Moved the GPS to the sensors sheet and removed the GPS sheet.
Other:
- removed sheet GPS
Changed lines of the file:
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@@
 	(paper "A4")
 	(sheet
-		(at 77.47 100.33)
+		(at 74.93 68.58)
 		(size 30.48 26.67)
 		(exclude_from_sim no)
@@
 		)
 		(property "Sheetname" "SD"
-			(at 77.47 99.6184 0)
+			(at 74.93 67.8684 0)
 			(effects
 				(font
@@
 		)
 		(property "Sheetfile" "basic_flight_controller_SD.kicad_sch"
-			(at 77.47 127.5846 0)
-			(effects
-				(font
-					(size 1.27 1.27)
-				)
-				(justify left top)
-			)
-		)
-		(instances
-			(project "flight-controller-basic"
-				(path "/e04fbe87-dc7c-407c-abef-b71ed1bbe06a"
-					(page "7")
-				)
-			)
-		)
-	)
-	(sheet
-		(at 34.29 100.33)
+			(at 74.93 95.8346 0)
+			(effects
+				(font
+					(size 1.27 1.27)
+				)
+				(justify left top)
+			)
+		)
+		(instances
+			(project "flight-controller-basic"
+				(path "/e04fbe87-dc7c-407c-abef-b71ed1bbe06a"
+					(page "6")
+				)
+			)
+		)
+	)
+	(sheet
+		(at 34.29 68.58)
 		(size 29.21 26.67)
 		(exclude_from_sim no)
@@
 		)
 		(property "Sheetname" "SENSORS"
-			(at 34.29 99.6184 0)
+			(at 34.29 67.8684 0)
 			(effects
 				(font
@@
 		)
 		(property "Sheetfile" "sensors.kicad_sch"
-			(at 34.29 127.5846 0)
-			(effects
-				(font
-					(size 1.27 1.27)
-				)
-				(justify left top)
-			)
-		)
-		(instances
-			(project "flight-controller-basic"
-				(path "/e04fbe87-dc7c-407c-abef-b71ed1bbe06a"
-					(page "4")
-				)
-			)
-		)
-	)
-	(sheet
-		(at 77.47 66.04)
+			(at 34.29 95.8346 0)
+			(effects
+				(font
+					(size 1.27 1.27)
+				)
+				(justify left top)
+			)
+		)
+		(instances
+			(project "flight-controller-basic"
+				(path "/e04fbe87-dc7c-407c-abef-b71ed1bbe06a"
+					(page "3")
+				)
+			)
+		)
+	)
+	(sheet
+		(at 76.2 35.56)
 		(size 31.75 24.13)
 		(exclude_from_sim no)
@@
 		)
 		(property "Sheetname" "RADIO"
-			(at 77.47 65.3284 0)
+			(at 76.2 34.8484 0)
 			(effects
 				(font
@@
 		)
 		(property "Sheetfile" "RADIO_G/RADIO_G.kicad_sch"
-			(at 77.47 90.7546 0)
-			(effects
-				(font
-					(size 1.27 1.27)
-				)
-				(justify left top)
-			)
-		)
-		(instances
-			(project "flight-controller-basic"
-				(path "/e04fbe87-dc7c-407c-abef-b71ed1bbe06a"
-					(page "6")
+			(at 76.2 60.2746 0)
+			(effects
+				(font
+					(size 1.27 1.27)
+				)
+				(justify left top)
+			)
+		)
+		(instances
+			(project "flight-controller-basic"
+				(path "/e04fbe87-dc7c-407c-abef-b71ed1bbe06a"
+					(page "5")
 				)
 			)
@@
 	)
 	(sheet
-		(at 34.29 66.04)
-		(size 29.21 27.94)
-		(exclude_from_sim no)
-		(in_bom yes)
-		(on_board yes)
-		(dnp no)
-		(fields_autoplaced yes)
-		(stroke
-			(width 0.1524)
-			(type solid)
-		)
-		(fill
-			(color 0 0 0 0.0000)
-		)
-		(property "Sheetname" "GPS"
-			(at 34.29 65.3284 0)
-			(effects
-				(font
-					(size 1.27 1.27)
-				)
-				(justify left bottom)
-			)
-		)
-		(property "Sheetfile" "omnia_FC_2026/IMU_FC_G/GP_GPS/GP_GPS.kicad_sch"
-			(at 34.29 94.5646 0)
-			(effects
-				(font
-					(size 1.27 1.27)
-				)
-				(justify left top)
-			)
-		)
-		(instances
-			(project "flight-controller-basic"
-				(path "/e04fbe87-dc7c-407c-abef-b71ed1bbe06a"
-					(page "3")
-				)
-			)
-		)
-	)
-	(sheet
-		(at 77.47 33.02)
+		(at 34.29 102.87)
 		(size 29.21 25.4)
 		(exclude_from_sim no)
@@
 		)
 		(property "Sheetname" "USB-C"
-			(at 77.47 32.3084 0)
+			(at 34.29 102.1584 0)
 			(effects
 				(font
@@
 		)
 		(property "Sheetfile" "FC_USB-C_G/FC_USB-C_G.kicad_sch"
-			(at 77.47 59.0046 0)
-			(effects
-				(font
-					(size 1.27 1.27)
-				)
-				(justify left top)
-			)
-		)
-		(instances
-			(project "flight-controller-basic"
-				(path "/e04fbe87-dc7c-407c-abef-b71ed1bbe06a"
-					(page "5")
-				)
-			)
+			(at 34.29 128.8546 0)
+			(effects
+				(font
+					(size 1.27 1.27)
+				)
+				(justify left top)
+			)
+		)
+		(instances
+			(project "flight-controller-basic"
+				(path "/e04fbe87-dc7c-407c-abef-b71ed1bbe06a"
+					(page "4")
+				)
+			)

Commit message: fixing filepath typo
Other:
- sheet RADIO: file RADIO_G/RADIO_G.kicad_sch -> RADIO_G.kicad_sch
- sheet USB-C: file FC_USB-C_G/FC_USB-C_G.kicad_sch -> FC_USB-C_G.kicad_sch
Changed lines of the file:
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@@
 			)
 		)
-		(property "Sheetfile" "RADIO_G/RADIO_G.kicad_sch"
+		(property "Sheetfile" "RADIO_G.kicad_sch"
 			(at 76.2 60.2746 0)
 			(effects
@@
 			)
 		)
-		(property "Sheetfile" "FC_USB-C_G/FC_USB-C_G.kicad_sch"
+		(property "Sheetfile" "FC_USB-C_G.kicad_sch"
 			(at 34.29 128.8546 0)
 			(effects

Commit message: Fixed the second round of issues Sam gave us
Other:
- removed sheet USB-C
Changed lines of the file:
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@@
 			(project "flight-controller-basic"
 				(path "/e04fbe87-dc7c-407c-abef-b71ed1bbe06a"
-					(page "6")
+					(page "5")
 				)
 			)
@@
 			(project "flight-controller-basic"
 				(path "/e04fbe87-dc7c-407c-abef-b71ed1bbe06a"
-					(page "5")
+					(page "4")
 				)
 			)
@@
 				)
 			)
-		)
-	)
-	(sheet
-		(at 34.29 102.87)
-		(size 29.21 25.4)
-		(exclude_from_sim no)
-		(in_bom yes)
-		(on_board yes)
-		(dnp no)
-		(fields_autoplaced yes)
-		(stroke
-			(width 0.1524)
-			(type solid)
-		)
-		(fill
-			(color 0 0 0 0.0000)
-		)
-		(property "Sheetname" "USB-C"
-			(at 34.29 102.1584 0)
-			(effects
-				(font
-					(size 1.27 1.27)
-				)
-				(justify left bottom)
-			)
-		)
-		(property "Sheetfile" "FC_USB-C_G.kicad_sch"
-			(at 34.29 128.8546 0)
-			(effects
-				(font
-					(size 1.27 1.27)
-				)
-				(justify left top)
-			)
-		)
-		(instances
-			(project "flight-controller-basic"
-				(path "/e04fbe87-dc7c-407c-abef-b71ed1bbe06a"
-					(page "4")
-				)
-			)
