File: RADIO_G.kicad_sch (KiCad schematic)
At the start: 4 parts

Commit message: fixing filepath typo
Parts:
- renumbered C1 to C12, U1 to U6
Changed lines of the file:
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@@
 		(dnp no)
 		(fields_autoplaced yes)
-		(property "Reference" "C1"
+		(property "Reference" "C12"
 			(at 130.81 92.7099 0)
 			(effects
@@
 				)
 			)
-			(project ""
+			(project "flight-controller-basic"
 				(path "/e04fbe87-dc7c-407c-abef-b71ed1bbe06a/8f3c10af-0dfe-45e5-9dde-cd3bf089277e"
 					(reference "C12")
@@
 				)
 			)
+			(project "flight-controller-basic"
+				(path "/e04fbe87-dc7c-407c-abef-b71ed1bbe06a/8f3c10af-0dfe-45e5-9dde-cd3bf089277e"
+					(reference "C3")
+					(unit 1)
+				)
+			)
 		)
 	)
@@
 		(dnp no)
 		(fields_autoplaced yes)
-		(property "Reference" "#PWR01"
+		(property "Reference" "#PWR019"
 			(at 100.33 116.84 0)
 			(effects
@@
 				)
 			)
-			(project ""
+			(project "flight-controller-basic"
 				(path "/e04fbe87-dc7c-407c-abef-b71ed1bbe06a/8f3c10af-0dfe-45e5-9dde-cd3bf089277e"
 					(reference "#PWR019")
@@
 		(dnp no)
 		(fields_autoplaced yes)
-		(property "Reference" "U1"
+		(property "Reference" "U6"
 			(at 146.05 80.0099 0)
 			(effects
@@
 				)
 			)
-			(project ""
+			(project "flight-controller-basic"
 				(path "/e04fbe87-dc7c-407c-abef-b71ed1bbe06a/8f3c10af-0dfe-45e5-9dde-cd3bf089277e"
 					(reference "U6")
@@
 				)
 			)
+			(project "flight-controller-basic"
+				(path "/e04fbe87-dc7c-407c-abef-b71ed1bbe06a/8f3c10af-0dfe-45e5-9dde-cd3bf089277e"
+					(reference "#PWR04")
+					(unit 1)
+				)
+			)
 		)
 	)
@@
 		(dnp no)
 		(fields_autoplaced yes)
-		(property "Reference" "#PWR03"
+		(property "Reference" "#PWR017"
 			(at 100.33 87.63 0)
 			(effects
@@
 				)
 			)
-			(project ""
+			(project "flight-controller-basic"
 				(path "/e04fbe87-dc7c-407c-abef-b71ed1bbe06a/8f3c10af-0dfe-45e5-9dde-cd3bf089277e"
 					(reference "#PWR017")
@@
 				)
 			)
-		)
-	)
-	(sheet_instances
-		(path "/"
-			(page "1")
-		)
-	)
-	(embedded_fonts no)
+			(project "flight-controller-basic"
+				(path "/e04fbe87-dc7c-407c-abef-b71ed1bbe06a/8f3c10af-0dfe-45e5-9dde-cd3bf089277e"
+					(reference "C2")
+					(unit 1)
+				)
+			)
+		)
+	)
 )
