File: FC_USB-C_G.kicad_sch (KiCad schematic)
At the start: 4 parts, among them J1 USB_C_Receptacle_USB2.0_16P

Commit message: Fixed the Barometer capacitors
Changed lines of the file:
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@@
 		(dnp no)
 		(property "Reference" "R3"
-			(at 148.844 77.724 90)
+			(at 141.478 77.47 90)
 			(effects
 				(font
@@
 		)
 		(property "Value" "5.11K"
-			(at 148.844 80.264 90)
+			(at 141.478 80.01 90)
 			(effects
 				(font
@@
 		(dnp no)
 		(property "Reference" "R2"
-			(at 149.352 72.136 90)
+			(at 140.716 71.628 90)
 			(effects
 				(font
@@
 		)
 		(property "Value" "5.11K"
-			(at 149.352 74.676 90)
+			(at 141.224 74.422 90)
 			(effects
 				(font
